File: sashwat-mc-one-smd-without-programmer/sashwat-mc-one-smd.brd (EAGLE design)
At the start: 44 x 28 mm, 15 parts, among them Q1 16Hz, U1 ATMEGA328P-AU

Commit message: Completed SMD design
Parts:
- moved LED2 0.26 mm to (40.4, 3.45)
- moved R3 0.26 mm to (41.5, 6.88)
- moved JP3 0.26 mm to (22.0, 24.8)
- moved JP2 0.26 mm to (21.8, 3.07)
- moved JP4 0.26 mm to (4.19, 23.3)
- moved JP1 0.26 mm to (4.19, 6.88)
- moved R1 0.26 mm to (4.19, 14.5)
- moved LED1 0.26 mm to (4.19, 18.6)
- moved R2 0.26 mm to (8.00, 20.7)
- moved S1 0.26 mm to (10.0, 12.2)
- moved C1 0.26 mm to (41.9, 23.0)
- moved C3 0.26 mm to (39.4, 23.0)
- moved C2 0.26 mm to (39.1, 6.88)
- moved Q1 0.26 mm to (40.3, 15.0)
- moved U1 0.26 mm to (26.9, 13.2)
Routing:
- net VCC: track 74.4 -> 72.5 mm
Other:
- board text added: "100nF"
- board text added: "10K"
- board text added: "16Hz"
- board text added: "220Ω"
- board text added: "22pF"
- board text added: "A0"
- board text added: "A1"
- board text added: "A2"
- board text added: "A3"
- board text added: "A4"
- board text added: "A5"
- board text added: "A6"
- board text added: "A7"
- board text added: "Atmega328p-AU"
- board text added: "D0"
- board text added: "D1"
- board text added: "D10"
- board text added: "D11"
- board text added: "D12"
- board text added: "D13"
- board text added: "D2"
- board text added: "D3"
- board text added: "D4"
- board text added: "D5"
- board text added: "D6"
- board text added: "D7"
- board text added: "D8"
- board text added: "D9"
- board text added: "GND"
- board text added: "LED"
- board text added: "MC ONE SMD (WP)"
- board text added: "POWER LED"
- board text added: "RESET"
- board text added: "RX"
- board text added: "Switch"
- board text added: "TX"
- board text added: "VCC"
- board text added: "sashwat.in"
