File: sashwat-mc-one-without-programmer/sashwat-mc-one.brd (EAGLE design)
At the start: 68.1 x 32.2 mm, 13 parts, among them IC1 ATMEGA328-20P, J1 F-1X04-SIP-100-40, J2 F-1X12-SIP-100-32Y, J3 F-1X12-SIP-100-32Y, Q1 16 MHz

Commit message: Updated non smd design
Parts:
- moved C1 23.1 mm to (89.7, 27.4)
- moved C2 23.1 mm to (89.7, 5.84)
- moved C3 23.1 mm to (82.3, 26.7)
- moved IC1 23.1 mm to (65.0, 15.7)
- moved J2 23.1 mm to (65.0, 5.59)
- moved J3 23.1 mm to (65.0, 27.2)
- moved C5 23.1 mm to (43.7, 26.9)
- moved R1 23.1 mm to (27.2, 15.7)
- moved S1 23.1 mm to (33.3, 27.4)
- moved J1 23.1 mm to (40.9, 15.7)
- moved LED3 23.1 mm to (32.0, 6.10)
- moved R5 23.1 mm to (32.0, 15.7)
- moved Q1 23.1 mm to (89.2, 16.5)
Routing:
- added copper zone on layer 1, net N$8
